File: Board_Layouts/EAGLE_designs/alphanewt/alphanewt_v1.8/BatteryBoard.brd (EAGLE design)
At the start: 158.4 x 117.7 mm, 16 parts, among them X3 C-GRID-10-70553, X4 C-GRID-10-70553

Commit message: Major update to alphanewt 1.8. Almost done routing the logic board.
Changed lines of the file:
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@@
 <hole x="92.71" y="30.8" drill="3.2004"/>
 <hole x="17.78" y="30.8" drill="3.2004"/>
-<hole x="2.1844" y="34.864" drill="3.2004"/>
 <text x="19.1" y="-17.9" size="1.016" layer="51">ARD Hole</text>
 <text x="71.1" y="-13.1" size="1.016" layer="51">ARD Hole</text>
