File: Board_Layouts/EAGLE_designs/alphanewt/alphanewt_v1.8/alphanewt_v1.8.sch (EAGLE design)
At the start: 98 parts, among them IC1 LM386N-1, Q1 TIP41C, Q2 TIP41C, Q3 TIP41C, Q4 TIP41C, Q5 TIP41C, Q6 TIP41C, Q7 TIP41C, T1 2N3904, T2 2N3904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

Commit message: Final updates to AlphaNewt v1.8 for review (fully routed)
Connections:
- removed net BATT2_TS2: X1-3.S
- removed net GPS_RX: GPS.6
- removed net GPS_TX: GPS.5
- removed net S/A_PWR_OUT_RTN: X2-2.S
- net BATT_2_TS2: now also X1-3.S
- net RX1: now also GPS.5
- net S/A_PWR_RTN: now also X2-2.S
- net TX1: now also GPS.6
Other:
- note removed: "CAMERA CIRCUIT"
Changed lines of the file:
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@@
 <text x="-40.64" y="78.74" size="1.778" layer="91">X0 = USB_Comp</text>
 <text x="-40.64" y="60.96" size="1.778" layer="91">X1 = GPS</text>
-<text x="157.48" y="93.98" size="1.778" layer="91">CAMERA CIRCUIT</text>
 <rectangle x1="208.28" y1="53.34" x2="233.68" y2="88.9" layer="97"/>
 </plain>
@@
 <junction x="-45.72" y="60.96"/>
 </segment>
+<segment>
+<wire x1="86.36" y1="-5.08" x2="48.26" y2="-5.08" width="0.1524" layer="91"/>
+<label x="48.26" y="-5.08" size="1.778" layer="95" rot="R180" xref="yes"/>
+<pinref part="GPS" gate="G$1" pin="6"/>
+</segment>
 </net>
 <net name="RX1" class="0">
@@
 <pinref part="ARD_5" gate="G$1" pin="6"/>
 <junction x="-45.72" y="58.42"/>
+</segment>
+<segment>
+<label x="68.58" y="-2.54" size="1.778" layer="95" rot="R180" xref="yes"/>
+<pinref part="GPS" gate="G$1" pin="5"/>
+<wire x1="68.58" y1="-2.54" x2="86.36" y2="-2.54" width="0.1524" layer="91"/>
 </segment>
 </net>
@@
 <junction x="-104.14" y="66.04"/>
 </segment>
+<segment>
+<label x="88.9" y="124.46" size="1.778" layer="95" rot="R180" xref="yes"/>
+<wire x1="88.9" y1="124.46" x2="114.3" y2="124.46" width="0.1524" layer="91"/>
+<pinref part="X1" gate="-3" pin="S"/>
+<junction x="114.3" y="124.46"/>
+</segment>
 </net>
 <net name="PYRO_1_PWR_RTN" class="1">
@@
 <wire x1="81.28" y1="-68.58" x2="81.28" y2="-63.5" width="0.1524" layer="91"/>
 </segment>
+<segment>
+<pinref part="X2" gate="-2" pin="S"/>
+<wire x1="114.3" y1="91.44" x2="111.76" y2="91.44" width="0.1524" layer="91"/>
+<label x="111.76" y="91.44" size="1.778" layer="95" rot="R180" xref="yes"/>
+<junction x="114.3" y="91.44"/>
+</segment>
 </net>
 <net name="S/A_PWR_IN" class="1">
@@
 </segment>
 </net>
-<net name="GPS_RX" class="0">
-<segment>
-<wire x1="86.36" y1="-5.08" x2="48.26" y2="-5.08" width="0.1524" layer="91"/>
-<label x="48.26" y="-5.08" size="1.778" layer="95" rot="R180" xref="yes"/>
-<pinref part="GPS" gate="G$1" pin="6"/>
-</segment>
-</net>
 <net name="GPS_VBAT" class="0">
 <segment>
@@
 </segment>
 </net>
-<net name="C_PWR/MODE" class="0">
-<segment>
-<label x="165.1" y="88.9" size="1.778" layer="95" xref="yes"/>
-<wire x1="165.1" y1="88.9" x2="165.1" y2="91.44" width="0.1524" layer="91"/>
-</segment>
-</net>
 <net name="CAMERA_PWR" class="1">
 <segment>
@@
 </segment>
 </net>
-<net name="S/A_PWR_OUT_RTN" class="0">
-<segment>
-<pinref part="X2" gate="-2" pin="S"/>
-<wire x1="114.3" y1="91.44" x2="111.76" y2="91.44" width="0.1524" layer="91"/>
-<label x="111.76" y="91.44" size="1.778" layer="95" rot="R180" xref="yes"/>
-<junction x="114.3" y="91.44"/>
-</segment>
-</net>
-<net name="BATT2_TS2" class="0">
-<segment>
-<label x="88.9" y="124.46" size="1.778" layer="95" rot="R180" xref="yes"/>
-<wire x1="88.9" y1="124.46" x2="114.3" y2="124.46" width="0.1524" layer="91"/>
-<pinref part="X1" gate="-3" pin="S"/>
-<junction x="114.3" y="124.46"/>
-</segment>
-</net>
 <net name="1PPS" class="0">
 <segment>
@@
 </segment>
 </net>
-<net name="GPS_TX" class="0">
-<segment>
-<label x="68.58" y="-2.54" size="1.778" layer="95" rot="R180" xref="yes"/>
-<pinref part="GPS" gate="G$1" pin="5"/>
-<wire x1="68.58" y1="-2.54" x2="86.36" y2="-2.54" width="0.1524" layer="91"/>
-</segment>
-</net>
